File: BluetoothSpeaker.kicad_sch (KiCad schematic)
At the start: 36 parts, among them J1 KF301-2P 5.08mm, Q1 AO4407A, SW1 RESET, SW2 BOOT, U1 AP63203WU-7, U2 AP63205WU-7, U3 ESP32-WROOM-32E-N4

Commit message: feat: update amplifier output stage and add OLED interface
Parts:
- removed Q1: AO4407A, Package_SO:SO-8_3.9x4.9mm_P1.27mm, symbol BluetoothSpeaker_Symbols:AO4407A
- added C16: 100nF 16V, Package_TO_SOT_SMD:SOT-23-6, symbol Device:C
- added C17: 4.7uF, Package_TO_SOT_SMD:SOT-23-6, symbol Device:C
- added C18, C19, C20, C22, C24, C26: 100nF, Package_TO_SOT_SMD:SOT-23-6, symbol Device:C
- added C21, C23, C25: 10uF, Package_TO_SOT_SMD:SOT-23-6, symbol Device:C
- added C27, C28: 2.2uF, symbol Device:C
- added C29, C30: 2.2nF, symbol Device:C
- added C31, C34: 1nF / 50V, symbol Device:C
- added C32, C35: 100nF / 50V, symbol Device:C
- added C33, C36: 220uF / 25V, symbol Device:C
- added C37, C48, C49: 100nF, symbol Device:C
- added C38: 1uF, symbol Device:C
- added C39, C40, C41, C42: 220nF / 25V, symbol Device:C
- added C43, C44, C45, C46: 1uF / 25V, Capacitor_SMD:C_0805_2012Metric, symbol Device:C
- added C47: 1uF, Capacitor_SMD:C_0805_2012Metric, symbol Device:C
- added C50, C51, C52, C53: 680nF, symbol Device:C
- added J2: USB4105, Connector_USB:USB_C_Receptacle_GCT_USB4105-xx-A_16P_TopMnt_Horizontal, symbol Connector:USB_C_Receptacle_USB2.0_16P
- added J3: J3 RIGHT SPEAKER, symbol Connector_Generic:Conn_01x02
- added J4: J4 LEFT SPEAKER, symbol Connector_Generic:Conn_01x02
- added J5: Conn_01x04, symbol Connector_Generic:Conn_01x04
- added L3, L4, L5, L6: 10uH, symbol Device:L
- added Q1: AO4407A, AO4407A:SOIC127P600X175-8N, symbol AO4407A:AO4407A
- added Q2, Q3: MMBT3904, Package_TO_SOT_SMD:SOT-23, symbol Transistor_BJT:MMBT3904
- added R10: 1k, symbol Device:R
- added R11, R12: 10k, Package_TO_SOT_SMD:SOT-23, symbol Device:R
- added R13: 150k 1%, Package_TO_SOT_SMD:SOT-23, symbol Device:R
- added R14: 30k 1%, Package_TO_SOT_SMD:SOT-23, symbol Device:R
- added R15: 1k, Package_TO_SOT_SMD:SOT-23, symbol Device:R
- added R16, R5: 0R, Resistor_SMD:R_0805_2012Metric, symbol Device:R
- added R17, R18, R19: 33R, Package_TO_SOT_SMD:SOT-23, symbol Device:R
- added R20, R26, R28, R30: 10k, symbol Device:R
- added R21, R22: 470R, symbol Device:R
- added R23: 5.6k, symbol Device:R
- added R24: 51k, Capacitor_SMD:C_0201_0603Metric, symbol Device:R
- added R25: 24k, Capacitor_SMD:C_0201_0603Metric, symbol Device:R
- added R27, R29: 100k, symbol Device:R
- added R6, R7: 5.1k, symbol Device:R
- added R8: 22.1k, symbol Device:R
- added R9: 47.5k, symbol Device:R
- added TP10: DAC_R, Relay_THT:Relay_DPDT_Schrack-RT2-FormC_RM5mm, symbol Connector:TestPoint
- added TP11: DAC_L, Relay_THT:Relay_DPDT_Schrack-RT2-FormC_RM5mm, symbol Connector:TestPoint
- added TP6: GNDD, symbol Connector:TestPoint
- added TP7: BAT_SENSE, Relay_THT:Relay_DPDT_Schrack-RT2-FormC_RM5mm, symbol Connector:TestPoint
- added TP8: GNDA, symbol Connector:TestPoint
- added TP9: XSMT, Relay_THT:Relay_DPDT_Schrack-RT2-FormC_RM5mm, symbol Connector:TestPoint
- added U4: USBLC6-2SC6, Package_TO_SOT_SMD:SOT-23-6, symbol Power_Protection:USBLC6-2SC6
- added U5: CP2102N-A02-GQFN28, Package_DFN_QFN:QFN-28-1EP_5x5mm_P0.5mm_EP3.35x3.35mm, symbol Interface_USB:CP2102N-Axx-xQFN28
- added U6: PCM5102APW, Package_SO:TSSOP-20_4.4x6.5mm_P0.65mm, symbol Audio:PCM5102A
- added U7: TPA3116D2DAD, Package_SO:Texas_DAD0032A_HTSSOP-32_6.1x11mm_P0.65mm_TopEP3.71x3.81mm, symbol TPA3116D2:TPA3116D2DAD
- TP3: value GND -> GND3PWR
Connections:
- net +3V3: now also C17.2, C18.2, C20.2, C21.2, C22.2, C23.2, C24.1, C25.1, R10.2, R20.2, R27.1, R30.2, U5.6 (VDD), U5.7 (VREGIN), U6.1 (CPVDD), U6.20 (DVDD), U6.8 (AVDD)
- net BAT_FUSED: now also Q1.5, Q1.6, Q1.7, Q1.8
- net BAT_PROTECTED: now also C31.1, C32.1, C33.1, C34.1, C35.1, C36.1, C37.1, Q1.1, Q1.2, Q1.3, R13.1, U7.17 (AVCC), U7.18 (PVCC), U7.19 (PVCC), U7.31 (PVCC), U7.32 (PVCC)
- net I2S_LRCK: now reaches U3.10 (IO25)
- net I2S_LRCK: now also R17.1
- net I2S_BCK: now reaches U3.11 (IO26)
- net I2S_BCK: now also R19.1
- net WS2812_DATA: now reaches U3.12 (IO27)
- net BTN_NEXT: now reaches U3.13 (IO14)
- net BTN_PREV: now reaches U3.16 (IO13)
- net STATUS_LED: now reaches R4.1, U3.24 (IO2)
- net ESP_IO0: now reaches R3.2, SW2.1, U3.25 (IO0)
- net ESP_IO0: now also Q3.3 (C)
- net AMP_MUTE: now reaches U3.27 (IO16)
- net AMP_MUTE: now also R26.1
- net AMP_SD: now reaches U3.28 (IO17)
- net AMP_SD: now also R28.2
- net ESP_EN: now reaches C15.1, R2.2, SW1.1, U3.3 (EN)
- net ESP_EN: now also Q2.3 (C)
- net ENC_SW: now reaches U3.30 (IO18)
- net I2S_DATA: now reaches U3.31 (IO19)
- net I2S_DATA: now also R18.1
- net OLED_SDA: now reaches U3.33 (IO21)
- net UART_RX: now reaches U3.34 (RXD0/IO3)
- net UART_RX: now also U5.26 (TXD)
- net UART_TX: now reaches U3.35 (TXD0/IO1)
- net UART_TX: now also U5.25 (RXD)
- net OLED_SCL: now reaches U3.36 (IO22)
- net BTN_BT: now reaches U3.37 (IO23)
- net BAT_SENSE: now reaches U3.6 (IO34)
- net BAT_SENSE: now also C19.1, R15.2, TP7.1
- net AMP_FAULT: now reaches U3.7 (IO35)
- net AMP_FAULT: now also R30.1, U7.3 (FAULTZ)
- net ENC_A: now reaches U3.8 (IO32)
- net ENC_B: now reaches U3.9 (IO33)
- net at R1.1: now also Q1.4
- net GND renamed GNDPWR
- net GNDPWR: now also C31.2, C32.2, C33.2, C34.2, C35.2, C36.2, C37.2, C38.1, C47.1, C48.2, C49.1, C50.2, C51.2, C52.2, C53.2, R23.2, R25.1, R29.2, R5.2, U7.1 (MODSEL), U7.13 (AM2), U7.14 (AM1), U7.15 (AM0), U7.22 (GND), U7.25 (GND), U7.28 (GND), U7.9 (GND); no longer C13.1, C14.1, C15.2, D2.1 (K), SW1.2, SW2.2, U3.[1,15,38,39] (GND)
- new net: R10.1, U5.9 (~{RST})
- new net: C42.1, L3.1, U7.21 (OUTNL)
- new net: C48.1, R26.2, R27.2, U7.12 (MUTE)
- new net: C40.1, L5.1, U7.27 (OUTNR)
- new net: R8.2, R9.2, U5.8 (VBUS)
- new net: J2.A5 (CC1), R6.2
- new net: J2.B5 (CC2), R7.2
- new net: C38.2, R24.2, U7.7 (GVDD)
- new net: Q2.1 (B), R11.2
- new net: R19.2, U6.13 (BCK)
- new net: R18.2, U6.14 (DIN)
- new net: R17.2, U6.15 (LRCK)
- new net: R20.1, TP9.1, U6.17 (XSMT)
- new net: C26.1, U6.18 (LDOO)
- new net: C27.1, U6.2 (CAPP)
- new net: C27.2, U6.4 (CAPM)
- new net: C28.1, U6.5 (VNEG)
- new net: R21.1, U6.6 (OUTL)
- new net: R22.1, U6.7 (OUTR)
- new net: Q3.1 (B), R12.2
- new net: C43.2, U7.10 (LINP)
- new net: C44.2, U7.11 (LINN)
- new net: C49.2, R28.1, R29.1, U7.2 (SDZ)
- new net: C42.2, U7.20 (BSNL)
- new net: C41.2, L4.1, U7.23 (OUTPL)
- new net: C41.1, U7.24 (BSPL)
- new net: C40.2, U7.26 (BSNR)
- new net: C39.1, L6.1, U7.29 (OUTPR)
- new net: C39.2, U7.30 (BSPR)
- new net: C45.2, U7.4 (RINP)
- new net: C46.2, U7.5 (RINN)
- new net: C47.2, R24.1, R25.2, U7.6 (PLIMIT)
- new net: R23.1, U7.8 (GAIN/SLV)
- new net ADC_BAT_RAW: R13.2, R14.1, R15.1
- new net CP_DTR: Q3.2 (E), R11.1, U5.28 (~{DTR})
- new net CP_RTS: Q2.2 (E), R12.1, U5.24 (~{RTS})
- new net DAC_L: C29.2, C43.1, R21.2, TP11.1
- new net DAC_R: C30.1, C45.1, R22.2, TP10.1
- new net GNDA: C20.1, C21.1, C24.2, C25.2, C28.2, C29.1, C30.2, C44.1, C46.1, R16.2, TP8.1, U6.3 (CPGND), U6.9 (AGND)
- new net GNDD: C13.1, C14.1, C15.2, C16.2, C17.1, C18.1, C19.2, C22.1, C23.1, C26.2, D2.1 (K), J2.A1 (GND), J2.A12 (GND), J2.B1 (GND), J2.B12 (GND), R14.2, R16.1, R5.1, R6.1, R7.1, R9.1, SW1.2, SW2.2, TP6.1, U3.[1,15,38,39] (GND), U4.2 (GND), U5.29 (GND), U5.3 (GND), U6.10 (DEMP), U6.11 (FLT), U6.12 (SCK), U6.16 (FMT), U6.19 (DGND)
- new net L+: C51.1, J4.1 (Pin_1), L4.2
- new net L-: C50.1, J4.2 (Pin_2), L3.2
- new net R+: C53.1, J3.1 (Pin_1), L6.2
- new net R-: C52.1, J3.2 (Pin_2), L5.2
- new net USB_DN: J2.A7 (D-), J2.B7 (D-), U4.4 (I/O2)
- new net USB_DN_ESD: U4.3 (I/O2), U5.5 (D-)
- new net USB_DP: J2.A6 (D+), J2.B6 (D+), U4.6 (I/O1)
- new net USB_DP_ESD: U4.1 (I/O1), U5.4 (D+)
- new net USB_SHIELD: J2.SH (SHIELD)
- new net USB_VBUS: C16.1, J2.A4 (VBUS), J2.A9 (VBUS), J2.B4 (VBUS), J2.B9 (VBUS), R8.1, U4.5 (VBUS)
- no-connect marks 0 -> 25
Other:
- note added: "3.3 V BUCK"
- note added: "5 V BUCK"
- note added: "AUDIO / AMPLIFIER"
- note added: "AUDIO / DAC"
- note added: "BATTERY MEASUREMENT"
- note added: "DIGITAL / ESP32 CORE"
- note added: "GROUND LINK"
- note added: "GROUND LINK - AUDIO"
- note added: "POWER"
- note added: "POWER INPUT & PROTECTION"
- note added: "USB / PROGRAMMING"
- note added: "USER INTERFACE / OLED"
- moved on the sheet: C1, C10, C11, C12, C13, C14, C15, C2, C3, C4, C5, C6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

Commit message: feat: add user interface controls and finalize speaker outputs
Parts:
- added J6: Conn_01x10, Connector_PinHeader_2.54mm:PinHeader_1x10_P2.54mm_Vertical, symbol Connector_Generic:Conn_01x10
- added R31, R32: 4.7k, symbol Device:R
- added R33, R34, R35, R36, R37, R38: 10k, symbol Device:R
- added R39, R40, R41, R42, R43, R44: 100R, symbol Device:R
- J5: footprint (none) -> Connector_PinHeader_2.54mm:PinHeader_1x04_P2.54mm_Vertical
Connections:
- net +3V3: now also J5.2 (Pin_2), J6.9 (Pin_9), R31.1, R32.1, R33.1, R34.1, R35.1, R36.1, R37.1, R38.2
- net BAT_FUSED: now also D1.2 (A)
- net BAT_PROTECTED: no longer D1.1 (K)
- net BTN_BT: now also R39.1
- net BTN_NEXT: now also R40.2
- net BTN_PREV: now also R41.2
- net ENC_A: now also R44.2
- net ENC_B: now also R43.1
- net ENC_SW: now also R42.1
- net GNDD: now also J5.1 (Pin_1), J6.1 (Pin_1), J6.10 (Pin_10), J6.5 (Pin_5)
- net GNDPWR: now also D1.1 (K); no longer D1.2 (A)
- net OLED_SCL: now also J5.4 (Pin_4), R31.2
- net OLED_SDA: now also J5.3 (Pin_3), R32.2
- new net: J6.4 (Pin_4), R35.2, R42.2
- new net: J6.8 (Pin_8), R37.2, R39.2
- new net: J6.3 (Pin_3), R34.2, R43.2
- new net: J6.2 (Pin_2), R33.2, R44.1
- new net: J6.6 (Pin_6), R36.2, R41.1
- new net: J6.7 (Pin_7), R38.1, R40.1
Other:
- note added: "USER INTERFACE / CONTROLS"
- moved on the sheet: J5

Commit message: Complete schematic ERC and WS2812 interface
Parts:
- added C54: 100nF, symbol Device:C
- added C55: 4.7uF, Package_TO_SOT_SMD:SOT-23-6, symbol Device:C
- added C56: 100nF, Package_TO_SOT_SMD:SOT-23-6, symbol Device:C
- added C57: 100nF, Capacitor_SMD:C_0805_2012Metric, symbol Device:C
- added C58: 100pF, symbol Device:C
- added J7: Conn_01x03, Connector_PinHeader_2.54mm:PinHeader_1x03_P2.54mm_Vertical, symbol Connector_Generic:Conn_01x03
- added R45: 100k, symbol Device:R
- added R46: 330R, Resistor_SMD:R_0805_2012Metric, symbol Device:R
- added R47: 1M, symbol Device:R
- added TP12: USB_3V3, symbol Connector:TestPoint
- added TP13: TP_I2S_DATA, symbol Connector:TestPoint
- added TP14: TP_I2S_LRCK, symbol Connector:TestPoint
- added TP15: TP_I2S_BCK, symbol Connector:TestPoint
- added TP16: TP_ESP_IO0, symbol Connector:TestPoint
- added TP17: TP_ESP_EN, symbol Connector:TestPoint
- added TP18: TP_AMP_MUTE, symbol Connector:TestPoint
- added TP19: TP_AMP_FAULT, symbol Connector:TestPoint
- added TP20: TP_AMP_SD, symbol Connector:TestPoint
- added U8: 74LVC2G126DCTRG4, SN74LVC2G126:DCT8, symbol SN74LVC2G126:74LVC2G126DCTRG4
- added U9: 74AHCT125, symbol 74xx:74AHCT125
- R11, R12: footprint Package_TO_SOT_SMD:SOT-23 -> Resistor_SMD:R_0805_2012Metric
- TP3: value GND3PWR -> GNDPWR
Connections:
- net +3V3: now also C54.2, U8.8 (VCC); no longer C17.2, C18.2, R10.2, U5.6 (VDD), U5.7 (VREGIN)
- net +5V: now also C57.2, J7.1 (Pin_1), U9.10, U9.13, U9.14 (VCC), U9.4
- net AMP_FAULT: now also TP19.1
- net AMP_MUTE: now also TP18.1
- net AMP_SD: now also TP20.1
- net ESP_EN: now also TP17.1
- net ESP_IO0: now also TP16.1
- net GNDD: now also C54.1, C55.1, C56.1, C57.1, C58.1, J7.3 (Pin_3), R45.1, R47.1, U8.4 (GND), U9.1, U9.12, U9.5, U9.7 (GND), U9.9
- net I2S_BCK: now also TP15.1
- net I2S_DATA: now also TP13.1
- net I2S_LRCK: now also TP14.1
- net UART_RX: now also U8.3 (2Y); no longer U5.26 (TXD)
- net UART_TX: now also U8.2 (1A); no longer U5.25 (RXD)
- net USB_SHIELD: now also C58.2, R47.2
- net USB_VBUS: now also U5.7 (VREGIN), C55.2, C56.2
- net WS2812_DATA: now also U9.2
- new net: U5.25 (RXD), U8.6 (1Y)
- new net: U5.26 (TXD), U8.5 (2A)
- new net: R46.1, U9.3
- new net USB_3V3: C17.2, C18.2, R10.2, R45.2, TP12.1, U5.6 (VDD), U8.1 (1OE), U8.7 (2OE)
- new net WS2812_DATA_5V: J7.2 (Pin_2), R46.2
- no-connect marks 25 -> 28
Other:
- note added: "USER INTERFACE / LEVEL SHIFTER"
- moved on the sheet: C15, C16, C17, C18, J2, Q2, Q3, R10, R11, R12, R2, R3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

Commit message: footprints
Parts:
- C1, C11, C12, C3, C50, C51, C52, C53, C6, C7, C9: footprint (none) -> Capacitor_SMD:C_1210_3225Metric
- C10, C14, C15, C2, C27, C28, C29, C30, C31, C32, C34, C35, C37, C38, C39, C4, C40, C41, C42, C48, C49, C5, C54, C8: footprint (none) -> Capacitor_SMD:C_0805_2012Metric
- C13, C58: footprint (none) -> Capacitor_SMD:C_1206_3216Metric
- C16, C17, C18, C19, C20, C22, C24, C26, C55, C56: footprint Package_TO_SOT_SMD:SOT-23-6 -> Capacitor_SMD:C_0805_2012Metric
- C21, C23, C25: footprint Package_TO_SOT_SMD:SOT-23-6 -> Capacitor_SMD:C_1206_3216Metric
- C33, C36: footprint (none) -> Capacitor_THT:CP_Radial_D8.0mm_P3.50mm
- D1: footprint (none) -> Diode_SMD:D_SMB
- D2: footprint (none) -> LED_SMD:LED_0805_2012Metric
- L1: footprint (none) -> Wurth_WE-CHSAP:L_Wurth_WE-CHSAP-8090
- L2, L3, L4, L5, L6: footprint (none) -> KiCad_WE-PD:L_Wurth_WE-PD-1050P
- R1, R10, R2, R20, R21, R22, R23, R26, R27, R28, R29, R3, R30, R31, R32, R33, R34, R35, R36, R37, R38, R39, R4, R40, R41, R42, R43, R44, R45, R47, R6, R7, R8, R9: footprint (none) -> Resistor_SMD:R_0805_2012Metric
- R13, R14, R15, R17, R18, R19: footprint Package_TO_SOT_SMD:SOT-23 -> Resistor_SMD:R_0805_2012Metric
- R24, R25: footprint Capacitor_SMD:C_0201_0603Metric -> Resistor_SMD:R_0805_2012Metric
- SW1: footprint Button_Switch_SMD:SW_SPST_PTS645 -> Button_Switch_THT:SW_PUSH_6mm
- SW2: footprint (none) -> Button_Switch_THT:SW_PUSH_6mm
- TP1, TP12, TP13, TP14, TP15, TP16, TP17, TP18, TP19, TP2, TP20, TP3, TP4, TP5, TP6, TP8: footprint (none) -> TestPoint:TestPoint_THTPad_D2.0mm_Drill1.0mm
- TP10, TP11, TP7, TP9: footprint Relay_THT:Relay_DPDT_Schrack-RT2-FormC_RM5mm -> TestPoint:TestPoint_THTPad_D2.0mm_Drill1.0mm
- U9: footprint (none) -> Package_SO:SOIC-14_3.9x8.7mm_P1.27mm

Commit message: feat: finalize schematic and initialize PCB layout
Parts:
- removed C33, C36: 220uF / 25V, Capacitor_THT:CP_Radial_D8.0mm_P3.50mm, symbol Device:C
- removed U8: 74LVC2G126DCTRG4, SN74LVC2G126:DCT8, symbol SN74LVC2G126:74LVC2G126DCTRG4
- added C33, C36: 220uF / 25V, Capacitor_THT:CP_Radial_D8.0mm_P3.50mm, symbol Device:C_Polarized
- added C59: 100nF, Capacitor_SMD:C_0805_2012Metric, symbol Device:C
- added U10, U11: 74LVC1G126, Package_TO_SOT_SMD:SOT-353_SC-70-5, symbol 74xGxx:74LVC1G126
- C50, C51, C52, C53: footprint Capacitor_SMD:C_1210_3225Metric -> Capacitor_SMD:C_1812_4532Metric
- F1: footprint (none) -> Capacitor_SMD:C_1808_4520Metric
- J1: value KF301-2P 5.08mm -> KLS2-300-5.00-02P-2S; footprint (none) -> TerminalBlock:TerminalBlock_MaiXu_MX126-5.0-02P_1x02_P5.00mm
- J3, J4: footprint (none) -> TerminalBlock:TerminalBlock_MaiXu_MX126-5.0-02P_1x02_P5.00mm
- L1: value 3.9uH -> 4.7uH; footprint Wurth_WE-CHSAP:L_Wurth_WE-CHSAP-8090 -> Inductor_SMD:L_Bourns_SRR1260
- L2, L3, L4, L5, L6: footprint KiCad_WE-PD:L_Wurth_WE-PD-1050P -> Inductor_SMD:L_Bourns_SRR1260
- U5: symbol Interface_USB:CP2102N-Axx-xQFN28 -> BluetoothSpeaker_Custom:CP2102N-Axx-xQFN28_Custom
- U7: symbol TPA3116D2:TPA3116D2DAD -> BluetoothSpeaker_Custom:TPA3116D2DAD_Custom
Connections:
- net +3V3: now also C54.1, C59.1, U10.5 (VCC), U11.5 (VCC); no longer C54.2
- net BAT_FUSED: now also D1.1 (K); no longer D1.2 (A)
- net BAT_PROTECTED: now also C33.1, C36.1
- net GNDD: now also C54.2, C59.2, U10.3 (GND), U11.3 (GND); no longer C54.1
- net GNDPWR: now also D1.2 (A), C33.2, C36.2; no longer D1.1 (K)
- net UART_RX: now also U11.4
- net UART_TX: now also U10.2
- net USB_3V3: now also U10.1, U11.1
- net at U5.25 (RXD): now also U10.4
- net at U5.26 (TXD): now also U11.2
Other:
- moved on the sheet: D1
